File: supply.kicad_sch (KiCad schematic)
At the start: 32 parts

Commit message: power good signal inversion && added part numbers
Parts:
- removed C?: 1u, symbol Device:C_Small
- removed C?: 47u, symbol Device:C_Small
- removed C?: 0.1u, symbol Device:C_Small
- removed C? (x2): 10u, symbol Device:C_Small
- removed L?: 1.5u, symbol Device:L_Small
- removed TP? (x3): TestPoint, symbol Connector:TestPoint
- added C? (x2): 10u/6.3V, Capacitor_SMD:C_0603_1608Metric_Pad1.08x0.95mm_HandSolder, symbol Device:C_Small
- added C?: 47u/6.3V, Capacitor_SMD:C_0603_1608Metric_Pad1.08x0.95mm_HandSolder, symbol Device:C_Small
- added C?: 100n/25V, Capacitor_SMD:C_0603_1608Metric_Pad1.08x0.95mm_HandSolder, symbol Device:C_Small
- added C?: 1u/10V, Capacitor_SMD:C_0603_1608Metric_Pad1.08x0.95mm_HandSolder, symbol Device:C_Small
- added L?: 1.5u/2.4A, Inductor_SMD:L_1008_2520Metric_Pad1.43x2.20mm_HandSolder, symbol Device:L_Small
- added Q?: Q_NPN_BEC, supply:TO-236AB, symbol Device:Q_NPN_BEC
- added R?: 47k, Resistor_SMD:R_0603_1608Metric_Pad0.98x0.95mm_HandSolder, symbol Device:R_Small
- added R?: 3k3, Resistor_SMD:R_0603_1608Metric_Pad0.98x0.95mm_HandSolder, symbol Device:R_Small
- added TP? (x3): TestPoint, TestPoint:TestPoint_Plated_Hole_D2.0mm, symbol Connector:TestPoint
- C?: value 10u -> 10u/6.3V; footprint (none) -> Capacitor_SMD:C_0603_1608Metric_Pad1.08x0.95mm_HandSolder; MNR (none) -> 187-CL10A106MQ8NNNC
- C?: value 22u -> 22u/6.3V; footprint (none) -> Capacitor_SMD:C_0603_1608Metric_Pad1.08x0.95mm_HandSolder; MNR (none) -> 81-GRM188R60J226ME5J
- C?: value 1u -> 1u/10V; footprint (none) -> Capacitor_SMD:C_0603_1608Metric_Pad1.08x0.95mm_HandSolder; MNR (none) -> 187-CL10A105KP8NNWC
- C?: value 22n -> 22n/50V; footprint (none) -> Capacitor_SMD:C_0603_1608Metric_Pad1.08x0.95mm_HandSolder; MNR (none) -> 603-CC603KPX7R9BB223
- C?: value 47u -> 47u/6.3V; footprint (none) -> Capacitor_SMD:C_0603_1608Metric_Pad1.08x0.95mm_HandSolder; MNR (none) -> 81-GRM188R60J476ME5J
- C?: value 0.1u -> 100n/25V; footprint (none) -> Capacitor_SMD:C_0603_1608Metric_Pad1.08x0.95mm_HandSolder; MNR (none) -> 603-CC603KRX7R8BB104
- IC?: MNR (none) -> 968-IS9307IRTAANFZT7
- IC?: MNR (none) -> 968-ISL85003FRZ
- L?: value 1.5u -> 1.5u/2.4A; footprint (none) -> Inductor_SMD:L_1008_2520Metric_Pad1.43x2.20mm_HandSolder; MNR (none) -> 963-MAKK2520H1R5M
- R? (x9): footprint (none) -> Resistor_SMD:R_0603_1608Metric_Pad0.98x0.95mm_HandSolder
- R?: footprint (none) -> aResistor_SMD:R_0603_1608Metric_Pad0.98x0.95mm_HandSolder
- TP?: footprint (none) -> TestPoint:TestPoint_Plated_Hole_D2.0mm
Connections:
- net +1V2: now also C?.1, L?.2
- net +2V5: now also C?.1, TP?.1
- net +3V3: now also C?.1, TP?.1
- net +5V: now also C?.2, R?.2, TP?.1
- net GND: now also IC?.4 (ENLDO1), C?.2, C?.2, C?.2, C?.2, Q?.2 (E)
- net ISL8500_PG: now also R?.1; no longer R?.1, R?.1, R?.1
- net at IC?.4 (FB), R?.1, R?.1: now also C?.1
- net at IC?.13 (SW2): now also L?.1
- net at IC?.11 (VDD): now also C?.1
- new net: Q?.1 (B), R?.2
- new net PG: Q?.3 (C), R?.1, R?.1, R?.1, R?.1
- no-connect marks 2 -> 1
Other:
- note added: "power good signal inverter"
