File: supply.kicad_sch (KiCad schematic)
At the start: 36 parts, among them IC1 ISL85003FRZ, IC2 ISL9307IRTAANFZ-T7A, J1 Barrel_Jack, J2 Conn_01x02_Male, Q1 Q_NPN_BEC

Commit message: Added FPGA footprints
Parts:
- J1: footprint SamacSys_Parts:PJ063BH -> fpga:PJ063BH
Changed lines of the file:
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@@
     (property "Reference" "J1" (id 0) (at 33.02 62.23 0))
     (property "Value" "Barrel_Jack" (id 1) (at 33.02 64.77 0))
-    (property "Footprint" "SamacSys_Parts:PJ063BH" (id 2) (at 34.29 72.136 0)
+    (property "Footprint" "fpga:PJ063BH" (id 2) (at 34.29 72.136 0)
       (effects (font (size 1.27 1.27)) hide)
     )

Commit message: first layout steps
Parts:
- removed C2: 100n/25V, Capacitor_SMD:C_0603_1608Metric_Pad1.08x0.95mm_HandSolder, symbol Device:C_Small
- added C?: 1u/10V, Capacitor_SMD:C_0603_1608Metric_Pad1.08x0.95mm_HandSolder, symbol Device:C_Small
- added L4: 4.7u, Inductor_SMD:L_Taiyo-Yuden_NR-50xx, symbol Device:L_Small
Connections:
- net ISL8500_EN is gone; now on an unnamed net: IC1.3 (EN)
- net +5V: now also L4.2; no longer L1.2
- net GND: now also C?.2
- net at IC1.11 (VDD): now also C?.1
- net at C3.1, IC1.7 (PHASE_1), IC1.8 (PHASE_2): now also L4.1; no longer L1.1
Other:
- moved on the sheet: L1
Changed lines of the file:
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@@
   (junction (at 181.61 93.98) (diameter 0) (color 0 0 0 0)
+  )
+  (junction (at 52.07 58.42) (diameter 0) (color 0 0 0 0)
   )
   (junction (at 186.69 93.98) (diameter 0) (color 0 0 0 0)
@@
   )
   (wire (pts (xy 214.63 58.42) (xy 217.17 58.42))
+    (stroke (width 0) (type default) (color 0 0 0 0))
+  )
+  (wire (pts (xy 52.07 50.8) (xy 52.07 58.42))
     (stroke (width 0) (type default) (color 0 0 0 0))
   )
@@
     )
   )
-  (global_label "ISL8500_EN" (shape input) (at 52.07 50.8 180) (fields_autoplaced)
-    (effects (font (size 1.27 1.27)) (justify right))
-    (property "Intersheet References" "${INTERSHEET_REFS}" (id 0) (at 38.5293 50.7206 0)
-      (effects (font (size 1.27 1.27)) (justify right) hide)
-    )
-  )
   (global_label "ISL_3V3" (shape output) (at 241.3 40.64 0) (fields_autoplaced)
     (effects (font (size 1.27 1.27)) (justify left))
@@
     (pin "1")
   )
+  (symbol (lib_id "Device:C_Small") (at 77.47 34.29 0) (unit 1)
+    (in_bom yes) (on_board yes) (fields_autoplaced)
+    (property "Reference" "C?" (id 0) (at 80.01 33.0262 0)
+      (effects (font (size 1.27 1.27)) (justify left))
+    )
+    (property "Value" "1u/10V" (id 1) (at 80.01 35.5662 0)
+      (effects (font (size 1.27 1.27)) (justify left))
+    )
+    (property "Footprint" "Capacitor_SMD:C_0603_1608Metric_Pad1.08x0.95mm_HandSolder" (id 2) (at 77.47 34.29 0)
+      (effects (font (size 1.27 1.27)) hide)
+    )
+    (property "Datasheet" "~" (id 3) (at 77.47 34.29 0)
+      (effects (font (size 1.27 1.27)) hide)
+    )
+    (property "MNR" " 187-CL10A105KP8NNWC " (id 5) (at 77.47 34.29 0)
+      (effects (font (size 1.27 1.27)) hide)
+    )
+    (pin "1")
+    (pin "2")
+  )
   (symbol (lib_id "Device:R_Small") (at 156.21 63.5 90) (unit 1)
     (in_bom yes) (on_board yes)
@@
   )
   (symbol (lib_id "Device:R_Small") (at 101.6 58.42 0) (unit 1)
-    (in_bom yes) (on_board yes) (fields_autoplaced)
+    (in_bom yes) (on_board yes)
     (property "Reference" "R3" (id 0) (at 104.14 57.1499 0)
       (effects (font (size 1.27 1.27)) (justify left))
@@
     )
     (pin "1")
+  )
+  (symbol (lib_id "Device:L_Small") (at 100.33 71.12 90) (unit 1)
+    (in_bom yes) (on_board yes) (fields_autoplaced)
+    (property "Reference" "L4" (id 0) (at 100.33 66.04 90))
+    (property "Value" "4.7u" (id 1) (at 100.33 68.58 90))
+    (property "Footprint" "Inductor_SMD:L_Taiyo-Yuden_NR-50xx" (id 2) (at 100.33 71.12 0)
+      (effects (font (size 1.27 1.27)) hide)
+    )
+    (property "Datasheet" "~" (id 3) (at 100.33 71.12 0)
+      (effects (font (size 1.27 1.27)) hide)
+    )
+    (property "MNR" " 963-NR5040T4R7N " (id 5) (at 100.33 71.12 90)
+      (effects (font (size 1.27 1.27)) hide)
+    )
+    (pin "1")
+    (pin "2")
   )
   (symbol (lib_id "power:GND") (at 92.71 63.5 0) (unit 1)
@@
     (pin "2")
   )
-  (symbol (lib_id "Device:C_Small") (at 77.47 34.29 0) (unit 1)
-    (in_bom yes) (on_board yes)
-    (property "Reference" "C2" (id 0) (at 80.01 33.0262 0)
-      (effects (font (size 1.27 1.27)) (justify left))
-    )
-    (property "Value" "100n/25V" (id 1) (at 80.01 30.48 0)
-      (effects (font (size 1.27 1.27)) (justify left))
-    )
-    (property "Footprint" "Capacitor_SMD:C_0603_1608Metric_Pad1.08x0.95mm_HandSolder" (id 2) (at 77.47 34.29 0)
-      (effects (font (size 1.27 1.27)) hide)
-    )
-    (property "Datasheet" "~" (id 3) (at 77.47 34.29 0)
-      (effects (font (size 1.27 1.27)) hide)
-    )
-    (property "MNR" " 603-CC603KRX7R8BB104 " (id 5) (at 77.47 34.29 0)
-      (effects (font (size 1.27 1.27)) hide)
-    )
-    (pin "1")
-    (pin "2")
-  )
   (symbol (lib_id "Device:R_Small") (at 156.21 60.96 90) (unit 1)
     (in_bom yes) (on_board yes)
@@
     (pin "2")
   )
-  (symbol (lib_id "Device:L_Small") (at 100.33 71.12 90) (unit 1)
-    (in_bom yes) (on_board yes) (fields_autoplaced)
-    (property "Reference" "L1" (id 0) (at 100.33 66.04 90))
-    (property "Value" "4.7u" (id 1) (at 100.33 68.58 90))
-    (property "Footprint" "supply:NR5040T4R7N" (id 2) (at 100.33 71.12 0)
-      (effects (font (size 1.27 1.27)) hide)
-    )
-    (property "Datasheet" "~" (id 3) (at 100.33 71.12 0)
-      (effects (font (size 1.27 1.27)) hide)
-    )
-    (property "MNR" " 963-NR5040T4R7N " (id 5) (at 100.33 71.12 90)
-      (effects (font (size 1.27 1.27)) hide)
-    )
+  (symbol (lib_id "Device:L_Small") (at 118.11 96.52 90) (unit 1)
+    (in_bom yes) (on_board yes) (fields_autoplaced)
+    (property "Reference" "L1" (id 0) (at 118.11 91.44 90))
+    (property "Value" "4.7u" (id 1) (at 118.11 93.98 90))
+    (property "Footprint" "supply:NR5040T4R7N" (id 2) (at 118.11 96.52 0)
+      (effects (font (size 1.27 1.27)) hide)
+    )
+    (property "Datasheet" "~" (id 3) (at 118.11 96.52 0)
+      (effects (font (size 1.27 1.27)) hide)
+    )
+    (property "MNR" " 963-NR5040T4R7N " (id 5) (at 118.11 96.52 90)
+      (effects (font (size 1.27 1.27)) hide)
+    )

Commit message: supply layout review step
Parts:
- gave numbers to parts that had none: 1
Changed lines of the file:
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@@
   (symbol (lib_id "Device:C_Small") (at 77.47 34.29 0) (unit 1)
     (in_bom yes) (on_board yes) (fields_autoplaced)
-    (property "Reference" "C?" (id 0) (at 80.01 33.0262 0)
+    (property "Reference" "C2" (id 0) (at 80.01 33.0262 0)
       (effects (font (size 1.27 1.27)) (justify left))
     )

Commit message: changed testpoint footprints
Parts:
- TP1, TP2, TP3, TP4: footprint TestPoint:TestPoint_Plated_Hole_D2.0mm -> TestPoint:TestPoint_THTPad_D1.5mm_Drill0.7mm
Changed lines of the file:
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@@
       (effects (font (size 1.27 1.27)) (justify left))
     )
-    (property "Footprint" "TestPoint:TestPoint_Plated_Hole_D2.0mm" (id 2) (at 53.34 119.38 0)
+    (property "Footprint" "TestPoint:TestPoint_THTPad_D1.5mm_Drill0.7mm" (id 2) (at 53.34 119.38 0)
       (effects (font (size 1.27 1.27)) hide)
     )
@@
       (effects (font (size 1.27 1.27)) (justify left))
     )
-    (property "Footprint" "TestPoint:TestPoint_Plated_Hole_D2.0mm" (id 2) (at 53.34 143.51 0)
+    (property "Footprint" "TestPoint:TestPoint_THTPad_D1.5mm_Drill0.7mm" (id 2) (at 53.34 143.51 0)
       (effects (font (size 1.27 1.27)) hide)
     )
@@
       (effects (font (size 1.27 1.27)) (justify left))
     )
-    (property "Footprint" "TestPoint:TestPoint_Plated_Hole_D2.0mm" (id 2) (at 53.34 134.62 0)
+    (property "Footprint" "TestPoint:TestPoint_THTPad_D1.5mm_Drill0.7mm" (id 2) (at 53.34 134.62 0)
       (effects (font (size 1.27 1.27)) hide)
     )
@@
       (effects (font (size 1.27 1.27)) (justify left))
     )
-    (property "Footprint" "TestPoint:TestPoint_Plated_Hole_D2.0mm" (id 2) (at 53.34 127 0)
-      (effects (font (size 1.27 1.27)) hide)
-    )
+    (property "Footprint" "TestPoint:TestPoint_THTPad_D1.5mm_Drill0.7mm" (id 2) (at 53.34 127 0)
+      (effects (font (size 1.27 1.27)) hide)
+    )
