File: supply.kicad_sch (KiCad schematic)
At the start: 37 parts, among them IC1 ISL85003FRZ, IC2 ISL9307IRTAANFZ-T7A, J1 Barrel_Jack, J2 Conn_01x02_Male, Q1 Q_NPN_BEC

Commit message: update footprint of jack
Parts:
- J1: footprint fpga:PJ063BH -> supply:PJ063BH
Changed lines of the file:
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@@
     (property "Reference" "J1" (id 0) (at 33.02 62.23 0))
     (property "Value" "Barrel_Jack" (id 1) (at 33.02 64.77 0))
-    (property "Footprint" "fpga:PJ063BH" (id 2) (at 34.29 72.136 0)
+    (property "Footprint" "supply:PJ063BH" (id 2) (at 34.29 72.136 0)
       (effects (font (size 1.27 1.27)) hide)
     )
